File: electronics/vi_curve_tracer.sch (KiCad schematic (older format))
At the start: 64 parts, among them P1 CONN_01X05, P2 USB_OTG, P3 CONN_01X06, P4 CONN_01X06, P5 CONN_01X02, U1 MCP6004, U2 pic24f08km202, U3 ft230x

Commit message: Updated BOM items based on feedback from octopart, added fiducials to layout
Parts:
- U1: MPN MCP6L04T-I/ST -> MCP6L04T-E/ST
- U2: MPN PIC24FV16KM202 -> PIC24FV16KM202-I/SO
