File: kicad/vi_curve_tracer.kicad_pcb (KiCad board)
At the start: 2 copper layers, 60 x 37 mm, 70 parts, among them P1 CONN_01X05, P2 USB_OTG, P3 CONN_01X02, P4 CONN_01X06, P5 CONN_01X02, P6 CONN_01X01, P7 CONN_01X01, P8 CONN_01X01, P9 CONN_01X01, U1 MCP6004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

Commit message: Updated to v1.3
Parts:
- added FID2: fiducial, kicad_pcb:fiducial, F.Cu at (168.5, 101.3)
Other:
- board text added: "curve tracer v1.3"
- board text added: "scope"
- board text removed: "GND"
- board text removed: "curve tracer v1.2"
Changed lines of the file:
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@@
-(kicad_pcb (version 4) (host pcbnew 4.0.1-stable)
+(kicad_pcb (version 4) (host pcbnew 4.0.5)
   (general
     (links 135)
     (no_connects 0)
-    (area 166.193999 70.601 228.051 112.501001)
+    (area 166.193999 70.751 228.151 112.501001)
     (thickness 1.6)
-    (drawings 17)
+    (drawings 56)
     (tracks 557)
     (zones 0)
-    (modules 70)
+    (modules 71)
     (nets 44)
   )
@@
     (add_net ~MCLR)
   )
+  (module kicad_pcb:fiducial locked (layer F.Cu)
+    (at 168.529 101.346)
+    (fp_text reference FID2 (at 2.54 0 180) (layer F.SilkS)
+      (effects (font (size 1 1) (thickness 0.15)))
+    )
+    (fp_text value fiducial (at 0 0) (layer F.Fab) hide
+      (effects (font (size 1 1) (thickness 0.15)))
+    )
+    (pad 1 smd circle (at 0 0) (size 1.016 1.016) (layers F.Cu F.Mask)
+      (solder_mask_margin 1.016))
+  )
   (module kicad_pcb:CONN_1x1_CT3150 (layer B.Cu)
     (at 213.995 98.425)
@@
   (module fiducial locked (layer F.Cu)
     (at 224.409 86.106)
-    (fp_text reference FID1 (at 1.143 -3.175 90) (layer F.SilkS)
+    (fp_text reference FID1 (at -2.54 0 180) (layer F.SilkS)
       (effects (font (size 1 1) (thickness 0.15)))
     )
@@
   (module kicad_pcb:SM_0603 (layer F.Cu)
     (at 189.484 87.884)
-    (fp_text reference C2 (at -0.381 1.524) (layer F.SilkS)
+    (fp_text reference C2 (at 0 -1.397) (layer F.SilkS)
       (effects (font (size 1.016 0.889) (thickness 0.2032)))
     )
@@
   (module kicad_pcb:CONN_1x5_0.1in (layer F.Cu)
     (at 168.402 91.44 270)
-    (fp_text reference P1 (at -6.985 -0.127 360) (layer F.SilkS)
+    (fp_text reference P1 (at -7.112 0 360) (layer F.SilkS)
       (effects (font (size 1 1) (thickness 0.15)))
     )
@@
   (module kicad_pcb:SM_0603 (layer F.Cu)
     (at 171.45 87.63 270)
-    (fp_text reference R1 (at 2.159 -0.762 360) (layer F.SilkS)
+    (fp_text reference R1 (at 2.159 0 360) (layer F.SilkS)
       (effects (font (size 1.016 0.889) (thickness 0.2032)))
     )
@@
   (module kicad_pcb:SM_0603 (layer F.Cu)
     (at 188.214 81.788 270)
-    (fp_text reference C10 (at -2.032 -0.381 360) (layer F.SilkS)
+    (fp_text reference C10 (at -0.762 -2.032 360) (layer F.SilkS)
       (effects (font (size 1.016 0.889) (thickness 0.2032)))
     )
@@
   (module kicad_pcb:SM_0603 (layer F.Cu)
     (at 210.185 90.424)
-    (fp_text reference R14 (at 2.676 0.076) (layer F.SilkS)
+    (fp_text reference R14 (at 0 -1.524) (layer F.SilkS)
       (effects (font (size 1.016 0.889) (thickness 0.2032)))
     )
@@
   (module kicad_pcb:SM_0603 (layer F.Cu)
     (at 218.059 87.122)
-    (fp_text reference C16 (at 2.54 0.127) (layer F.SilkS)
+    (fp_text reference C16 (at 2.54 0.508) (layer F.SilkS)
       (effects (font (size 1.016 0.889) (thickness 0.2032)))
     )
@@
   (module kicad_pcb:SM_0603 (layer F.Cu)
     (at 218.059 88.773)
-    (fp_text reference C17 (at 2.54 0) (layer F.SilkS)
+    (fp_text reference C17 (at 2.54 0.381) (layer F.SilkS)
       (effects (font (size 1.016 0.889) (thickness 0.2032)))
     )
@@
   (module kicad_pcb:SM_0603 (layer F.Cu)
     (at 184.658 78.74 90)
-    (fp_text reference C20 (at 1.905 0 180) (layer F.SilkS)
+    (fp_text reference C20 (at 2.286 0 180) (layer F.SilkS)
       (effects (font (size 1.016 0.889) (thickness 0.2032)))
     )
@@
   (module kicad_pcb:SM_0603 (layer F.Cu)
     (at 186.182 78.74 90)
-    (fp_text reference C21 (at 0.762 2.032 180) (layer F.SilkS)
+    (fp_text reference C21 (at 0 2.032 180) (layer F.SilkS)
       (effects (font (size 1.016 0.889) (thickness 0.2032)))
     )
@@
   (module kicad_pcb:SM_0603 (layer F.Cu)
     (at 186.182 93.218 180)
-    (fp_text reference R18 (at -2.54 0 180) (layer F.SilkS)
+    (fp_text reference R18 (at -2.54 0.254 180) (layer F.SilkS)
       (effects (font (size 1.016 0.889) (thickness 0.2032)))
     )
@@
   (module kicad_pcb:SM_0603 (layer F.Cu)
     (at 181.61 78.74 270)
-    (fp_text reference R21 (at -2.286 0 360) (layer F.SilkS)
+    (fp_text reference R21 (at -2.286 -0.127 360) (layer F.SilkS)
       (effects (font (size 1.016 0.889) (thickness 0.2032)))
     )
@@
   (module kicad_pcb:fiducial locked (layer F.Cu)
     (at 224.409 101.346)
-    (fp_text reference FID2 (at 1.016 3.048 90) (layer F.SilkS)
+    (fp_text reference FID2 (at -2.54 0 180) (layer F.SilkS)
       (effects (font (size 1 1) (thickness 0.15)))
     )
@@
   (module lib_pcb:CONN_1x1_EDGE_SCOPE_GND (layer F.Cu)
     (at 196.215 110.236)
-    (fp_text reference P8 (at 3.556 0) (layer F.SilkS)
+    (fp_text reference P8 (at 3.683 0) (layer F.SilkS)
       (effects (font (size 1 1) (thickness 0.15)))
     )
@@
   (module lib_pcb:CONN_1x1_EDGE_SCOPE_GND (layer F.Cu)
     (at 188.595 110.236)
-    (fp_text reference P9 (at 3.556 0) (layer F.SilkS)
+    (fp_text reference P9 (at 3.683 0) (layer F.SilkS)
       (effects (font (size 1 1) (thickness 0.15)))
     )
@@
       (net 40 /x))
   )
+  (gr_line (start 202.438 109.601) (end 201.549 109.601) (angle 90) (layer B.SilkS) (width 0.2))
+  (gr_line (start 201.549 110.49) (end 202.438 109.601) (angle 90) (layer B.SilkS) (width 0.2))
+  (gr_line (start 200.66 109.601) (end 201.549 110.49) (angle 90) (layer B.SilkS) (width 0.2))
+  (gr_line (start 201.549 109.601) (end 200.66 109.601) (angle 90) (layer B.SilkS) (width 0.2))
+  (gr_line (start 201.549 108.331) (end 201.549 109.601) (angle 90) (layer B.SilkS) (width 0.2))
+  (gr_line (start 196.215 108.331) (end 201.549 108.331) (angle 90) (layer B.SilkS) (width 0.2))
+  (gr_line (start 196.215 108.331) (end 196.215 108.712) (angle 90) (layer B.SilkS) (width 0.2))
+  (gr_line (start 188.595 108.331) (end 196.215 108.331) (angle 90) (layer B.SilkS) (width 0.2))
+  (gr_line (start 188.595 108.712) (end 188.595 108.331) (angle 90) (layer B.SilkS) (width 0.2))
+  (gr_text Y (at 185.547 105.664) (layer B.SilkS)
+    (effects (font (size 1.5 1.5) (thickness 0.3)) (justify mirror))
+  )
+  (gr_text X (at 192.659 105.664) (layer B.SilkS)
+    (effects (font (size 1.5 1.5) (thickness 0.3)) (justify mirror))
+  )
+  (gr_line (start 184.658 104.013) (end 184.658 111.252) (angle 90) (layer B.SilkS) (width 0.2))
+  (gr_line (start 201.803 104.013) (end 208.915 111.125) (angle 90) (layer B.SilkS) (width 0.2))
+  (gr_line (start 184.658 104.013) (end 201.803 104.013) (angle 90) (layer B.SilkS) (width 0.2))
+  (gr_text scope (at 199.009 105.791) (layer B.SilkS)
+    (effects (font (size 1.5 1.5) (thickness 0.3)) (justify mirror))
+  )
+  (gr_line (start 181.229 105.41) (end 182.753 105.41) (angle 90) (layer F.SilkS) (width 0.2))
+  (gr_line (start 181.991 104.648) (end 181.991 105.41) (angle 90) (layer F.SilkS) (width 0.2))
+  (gr_line (start 180.086 104.648) (end 181.991 104.648) (angle 90) (layer F.SilkS) (width 0.2))
+  (gr_line (start 181.483 106.426) (end 180.34 106.426) (angle 90) (layer F.SilkS) (width 0.2))
+  (gr_line (start 181.991 106.426) (end 182.626 106.426) (angle 90) (layer F.SilkS) (width 0.2))
+  (gr_line (start 182.626 106.426) (end 182.88 106.426) (angle 90) (layer F.SilkS) (width 0.2))
+  (gr_line (start 182.626 105.791) (end 182.626 106.426) (angle 90) (layer F.SilkS) (width 0.2))
+  (gr_line (start 182.499 105.791) (end 182.753 105.791) (angle 90) (layer F.SilkS) (width 0.2))
+  (gr_line (start 181.991 105.791) (end 181.991 106.426) (angle 90) (layer F.SilkS) (width 0.2))
+  (gr_line (start 181.864 105.791) (end 182.118 105.791) (angle 90) (layer F.SilkS) (width 0.2))
+  (gr_line (start 181.229 105.791) (end 181.483 105.791) (angle 90) (layer F.SilkS) (width 0.2))
+  (gr_line (start 177.8 105.41) (end 177.8 106.426) (angle 90) (layer F.SilkS) (width 0.2))
+  (gr_line (start 179.324 105.41) (end 177.8 105.41) (angle 90) (layer F.SilkS) (width 0.2))
+  (gr_line (start 180.086 104.648) (end 179.324 105.41) (angle 90) (layer F.SilkS) (width 0.2))
+  (gr_line (start 182.88 106.426) (end 182.88 106.934) (angle 90) (layer F.SilkS) (width 0.2))
+  (gr_line (start 181.483 106.426) (end 181.483 105.791) (angle 90) (layer F.SilkS) (width 0.2))
+  (gr_line (start 180.34 106.934) (end 180.34 106.426) (angle 90) (layer F.SilkS) (width 0.2))
+  (gr_line (start 196.215 108.331) (end 196.215 108.712) (angle 90) (layer F.SilkS) (width 0.2))
+  (gr_line (start 206.375 108.331) (end 206.375 109.601) (angle 90) (layer F.SilkS) (width 0.2))
+  (gr_line (start 188.595 108.331) (end 206.375 108.331) (angle 90) (layer F.SilkS) (width 0.2))
+  (gr_line (start 188.595 108.712) (end 188.595 108.331) (angle 90) (layer F.SilkS) (width 0.2))
+  (gr_line (start 207.391 109.601) (end 206.375 109.601) (angle 90) (layer F.SilkS) (width 0.2))
+  (gr_line (start 206.375 110.617) (end 207.391 109.601) (angle 90) (layer F.SilkS) (width 0.2))
+  (gr_line (start 205.359 109.601) (end 206.375 110.617) (angle 90) (layer F.SilkS) (width 0.2))
+  (gr_line (start 206.375 109.601) (end 205.359 109.601) (angle 90) (layer F.SilkS) (width 0.2))
   (gr_text Y (at 185.547 105.664) (layer F.SilkS)
     (effects (font (size 1.5 1.5) (thickness 0.3)))
@@
     (effects (font (size 1.27 1.016) (thickness 0.254)))
   )
-  (gr_text GND (at 196.215 107.95) (layer F.SilkS)
-    (effects (font (size 1.27 1.016) (thickness 0.254)))
-  )
   (gr_text V- (at 200.406 98.425) (layer B.SilkS)
     (effects (font (size 1.27 1.016) (thickness 0.254)) (justify mirror))
@@
     (effects (font (size 1.27 1.143) (thickness 0.254)))
   )
-  (gr_text "curve tracer v1.2" (at 199.263 77.089) (layer F.SilkS)
+  (gr_text "curve tracer v1.3" (at 199.263 77.089) (layer F.SilkS)
     (effects (font (size 1.016 1.27) (thickness 0.254)))
   )
